Commit message: Mesh paths updated.

File: digit.urdf (robot description, URDF)
Before this commit: robot digit, 29 links, 28 joints
Links:
- link left_elbow: geometry collision mesh filename=package://DigitRobotURDF/meshes/arm-L4.dae; visual mesh filename=package://DigitRobotURDF/meshes/arm-L4.dae
- link left_hip_pitch: geometry collision mesh filename=package://DigitRobotURDF/meshes/hip-pitch.dae; visual mesh filename=package://DigitRobotURDF/meshes/hip-pitch.dae
- link left_hip_roll: geometry collision mesh filename=package://DigitRobotURDF/meshes/hip-yaw-housing.dae; visual mesh filename=package://DigitRobotURDF/meshes/hip-yaw-housing.dae
- link left_hip_yaw: geometry collision mesh filename=package://DigitRobotURDF/meshes/hip-pitch-housing.dae; visual mesh filename=package://DigitRobotURDF/meshes/hip-pitch-housing.dae
- link left_knee: geometry collision mesh filename=package://DigitRobotURDF/meshes/knee.dae; visual mesh filename=package://DigitRobotURDF/meshes/knee.dae
- link left_shin: geometry collision mesh filename=package://DigitRobotURDF/meshes/shin.dae; visual mesh filename=package://DigitRobotURDF/meshes/shin.dae
- link left_shoulder_cap: geometry collision mesh filename=package://DigitRobotURDF/meshes/shoulder-roll-housing.dae; visual mesh filename=package://DigitRobotURDF/meshes/shoulder-roll-housing.dae
- link left_shoulder_pitch: geometry collision mesh filename=package://DigitRobotURDF/meshes/arm-L2.dae; visual mesh filename=package://DigitRobotURDF/meshes/arm-L2.dae
- link left_shoulder_roll: geometry collision mesh filename=package://DigitRobotURDF/meshes/arm-L1.dae; visual mesh filename=package://DigitRobotURDF/meshes/arm-L1.dae
- link left_shoulder_yaw: geometry collision mesh filename=package://DigitRobotURDF/meshes/arm-L3.dae; visual mesh filename=package://DigitRobotURDF/meshes/arm-L3.dae
- link left_tarsus: geometry collision mesh filename=package://DigitRobotURDF/meshes/tarsus.dae; visual mesh filename=package://DigitRobotURDF/meshes/tarsus.dae
- link left_toe_pitch: geometry collision mesh filename=package://DigitRobotURDF/meshes/toe-pitch.dae; visual mesh filename=package://DigitRobotURDF/meshes/toe-pitch.dae
- link left_toe_roll: geometry collision mesh filename=package://DigitRobotURDF/meshes/toe-roll.dae; visual mesh filename=package://DigitRobotURDF/meshes/toe-roll.dae
- link left_waist_cap: geometry collision mesh filename=package://DigitRobotURDF/meshes/shoulder-roll-housing.dae; visual mesh filename=package://DigitRobotURDF/meshes/shoulder-roll-housing.dae
- link right_elbow: geometry collision mesh filename=package://DigitRobotURDF/meshes/arm-L4.dae scale=1 -1 1; visual mesh filename=package://DigitRobotURDF/meshes/arm-L4.dae scale=1 -1 1
- link right_hip_pitch: geometry collision mesh filename=package://DigitRobotURDF/meshes/hip-pitch.dae scale=1 -1 1; visual mesh filename=package://DigitRobotURDF/meshes/hip-pitch.dae scale=1 -1 1
- link right_hip_roll: geometry collision mesh filename=package://DigitRobotURDF/meshes/hip-yaw-housing.dae scale=1 -1 1; visual mesh filename=package://DigitRobotURDF/meshes/hip-yaw-housing.dae scale=1 -1 1
- link right_hip_yaw: geometry collision mesh filename=package://DigitRobotURDF/meshes/hip-pitch-housing.dae scale=1 -1 1; visual mesh filename=package://DigitRobotURDF/meshes/hip-pitch-housing.dae scale=1 -1 1
- link right_knee: geometry collision mesh filename=package://DigitRobotURDF/meshes/knee.dae scale=1 -1 1; visual mesh filename=package://DigitRobotURDF/meshes/knee.dae scale=1 -1 1
- link right_shin: geometry collision mesh filename=package://DigitRobotURDF/meshes/shin.dae scale=1 -1 1; visual mesh filename=package://DigitRobotURDF/meshes/shin.dae scale=1 -1 1
- link right_shoulder_cap: geometry collision mesh filename=package://DigitRobotURDF/meshes/shoulder-roll-housing.dae scale=1 -1 1; visual mesh filename=package://DigitRobotURDF/meshes/shoulder-roll-housing.dae scale=1 -1 1
- link right_shoulder_pitch: geometry collision mesh filename=package://DigitRobotURDF/meshes/arm-L2.dae scale=1 -1 1; visual mesh filename=package://DigitRobotURDF/meshes/arm-L2.dae scale=1 -1 1
- link right_shoulder_roll: geometry collision mesh filename=package://DigitRobotURDF/meshes/arm-L1.dae scale=1 -1 1; visual mesh filename=package://DigitRobotURDF/meshes/arm-L1.dae scale=1 -1 1
- link right_shoulder_yaw: geometry collision mesh filename=package://DigitRobotURDF/meshes/arm-L3.dae scale=1 -1 1; visual mesh filename=package://DigitRobotURDF/meshes/arm-L3.dae scale=1 -1 1
- link right_tarsus: geometry collision mesh filename=package://DigitRobotURDF/meshes/tarsus.dae scale=1 -1 1; visual mesh filename=package://DigitRobotURDF/meshes/tarsus.dae scale=1 -1 1
- link right_toe_pitch: geometry collision mesh filename=package://DigitRobotURDF/meshes/toe-pitch.dae scale=1 -1 1; visual mesh filename=package://DigitRobotURDF/meshes/toe-pitch.dae scale=1 -1 1
- link right_toe_roll: geometry collision mesh filename=package://DigitRobotURDF/meshes/toe-roll.dae scale=1 -1 1; visual mesh filename=package://DigitRobotURDF/meshes/toe-roll.dae scale=1 -1 1
- link right_waist_cap: geometry collision mesh filename=package://DigitRobotURDF/meshes/shoulder-roll-housing.dae scale=1 -1 1; visual mesh filename=package://DigitRobotURDF/meshes/shoulder-roll-housing.dae scale=1 -1 1
- link torso: geometry collision mesh filename=package://DigitRobotURDF/meshes/torso.dae; visual mesh filename=package://DigitRobotURDF/meshes/torso.dae
